Commit message: Update urdf

File: blindbuy_description/urdf/cart.urdf (robot description, URDF)
Before this commit: robot cart, 13 links, 12 joints
Links:
- added link al_profile
Joints:
- added joint al_profile_joint: type fixed, parent base_link, child al_profile, origin xyz=0.37 0 0.45 rpy=0 0 0
- joint oak-d_joint: origin xyz=0 0 0.1 rpy=0 0 0 -> xyz=0 0 0.1 rpy=0 0 -1.5708
- joint ptz_base_joint: origin xyz=0.35 0 1 rpy=0 0 0 -> xyz=0 0 0.5 rpy=0 0 0; parent base_link -> al_profile

Commit message: Update urdf

File: blindbuy_description/urdf/cart.urdf (robot description, URDF)
Before this commit: robot cart, 14 links, 13 joints
Links:
- link al_profile: geometry visual mesh filename=package://blindbuy_description/meshes/al_profile.dae scale=0.001 0.001 0.001
Joints:
- joint al_profile_joint: origin xyz=0.37 0 0.45 rpy=0 0 0 -> xyz=0.36 0 0.45 rpy=0 0 0
- joint oak-d_joint: origin xyz=0 0 0.1 rpy=0 0 -1.5708 -> xyz=-0.002 -0.018 0.101 rpy=0 0 -1.5708
- joint ptz_base_joint: origin xyz=0 0 0.5 rpy=0 0 0 -> xyz=0 0 0.65 rpy=0 0 0

Commit message: Add demo 1: pan and tilt tracker

File: blindbuy_description/urdf/cart.urdf (robot description, URDF)
Before this commit: robot cart, 14 links, 13 joints
Joints:
- removed joint ptz_pan_joint
- removed joint ptz_tilt_joint
- added joint ptz_pan: type revolute, parent ptz_base, child ptz_body, origin xyz=0 0 0.013 rpy=0 0 0, axis 0 0 1, limit lower=-3.1416 upper=3.1416 effort=10 velocity=3
- added joint ptz_tilt: type revolute, parent ptz_body, child ptz_head, origin xyz=0 0 0.035 rpy=0 0 0, axis 1 0 0, limit lower=-1.5708 upper=1.5708 effort=10 velocity=3
